Commit message: Update Pioneer navigation files

File: robots/pioneer.urdf (robot description, URDF)
Before this commit: robot pioneer3at_body, 18 links, 17 joints
Links:
- link laser_frame: geometry collision box size=0.01 0.01 0.01; visual mesh filename=/home/rahma/AUTOGRP3/robots/meshes/hokuyo1.dae

Commit message: Update pioneer URDF

File: robots/pioneer.urdf (robot description, URDF)
Before this commit: robot pioneer3at_body, 18 links, 17 joints
Joints:
- joint cam_joint: origin xyz=0.24 0 0.084 rpy=0 0 0 -> xyz=0.30 0 0.25 rpy=0 0 0

Commit message: Update urdf and waypoint

File: robots/pioneer.urdf (robot description, URDF)
Before this commit: robot pioneer3at_body, 18 links, 17 joints
Links:
- link laser_frame: geometry collision box size=0.01 0.01 0.01; visual mesh filename=/mnt/c/Users/Lithi/Desktop/AUTO4408/Project 1/AUTOGRP3/robo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

Commit message: Update Docker, Pioneer URDF, launch files, and control node configuration

File: robots/pioneer.urdf (robot description, URDF)
Before this commit: robot pioneer3at_body, 18 links, 17 joints
Links:
- link cam_frame: geometry visual box size=0.05 0.01 0.01
Joints:
- joint cam_joint: origin xyz=0.30 0 0.25 rpy=0 0 0 -> xyz=0.38 0 0.20 rpy=0 0 0
